File: KV1-pcb/KV1-pcb.kicad_pcb (KiCad board)
At the start: 2 copper layers, 0 parts

Commit message: Progressing on PCD design
Parts:
- added C1: 1uF, Capacitor_SMD:C_0805_2012Metric, B.Cu at (128.5, 74.4)
- added C2: 0.1uF, Capacitor_SMD:C_0805_2012Metric, B.Cu at (109.3, 81.8)
- added C3: 0.1uF, Capacitor_SMD:C_0805_2012Metric, B.Cu at (109.3, 78.4)
- added C4: 0.1uF, Capacitor_SMD:C_0805_2012Metric, B.Cu at (109.2, 71.5)
- added C5: 10uF, Capacitor_SMD:C_0805_2012Metric, B.Cu at (109.3, 74.7)
- added C6: 22pF, Capacitor_SMD:C_0805_2012Metric, B.Cu at (114.0, 85.0)
- added C7: 22pF, Capacitor_SMD:C_0805_2012Metric, B.Cu at (123.1, 85.0)
- added D1: D_Small, Diode_SMD:D_SOD-123, B.Cu at (146.3, 65.1)
- added D2: D_Small, Diode_SMD:D_SOD-123, B.Cu at (165.6, 65.0)
- added D3: D_Small, Diode_SMD:D_SOD-123, B.Cu at (146.6, 84.1)
- added D4: D_Small, Diode_SMD:D_SOD-123, B.Cu at (165.6, 84.1)
- added F1: 500mA, Fuse:Fuse_1206_3216Metric, B.Cu at (114.7, 60.4)
- added MX1: MX-NoLED, MX_Alps_Hybrid:MX-1U-NoLED, F.Cu at (138.1, 65.1)
- added MX2: MX-NoLED, MX_Alps_Hybrid:MX-1U-NoLED, F.Cu at (157.2, 65.1)
- added MX3: MX-NoLED, MX_Alps_Hybrid:MX-1U-NoLED, F.Cu at (138.1, 84.1)
- added MX4: MX-NoLED, MX_Alps_Hybrid:MX-1U-NoLED, F.Cu at (157.2, 84.1)
- added R1: 10k, Resistor_SMD:R_0805_2012Metric, B.Cu at (109.6, 65.8)
- added R2: 22, Resistor_SMD:R_0805_2012Metric, B.Cu at (119.5, 64.0)
- added R3: 22, Resistor_SMD:R_0805_2012Metric, B.Cu at (122.9, 64.0)
- added R4: 10k, Resistor_SMD:R_0805_2012Metric, B.Cu at (126.7, 83.8)
- added SW1: SW_Push, random-keyboard-parts:SKQG-1155865, B.Cu at (123.6, 91.2)
- added U1: ATmega32U4-A, Package_QFP:TQFP-44_10x10mm_P0.8mm, B.Cu at (119.1, 74.5)
- added USB1: Molex-0548190589, random-keyboard-parts:Molex-0548190589, B.Cu at (122.2, 53.9)
- added Y1: 16MHz, Crystal:Crystal_SMD_3225-4Pin_3.2x2.5mm, B.Cu at (118.4, 85.1)
